Commit message: 5

File: description/rl_scene_description/urdf/rl_scene.urdf (robot description, URDF)
Before this commit: robot rl_scene, 14 links, 13 joints
Joints:
- removed joint box_2_joint
- added joint grasp_point_joint: type fixed, parent panda_1_link8, child link_gripper, origin xyz=0.0 0.0 0.0 rpy=0 0 0

File: description/rl_scene_description/urdf/rl_scene.xacro (robot description, xacro)
@@ -108,6 +108,6 @@
   </joint>
   <!-- right arm with gripper -->
-  <xacro:panda_arm arm_id="$(arg arm_id_1)" connected_to="base_link"  xyz="0.0 0.0 0.0" safety_distance="0.03"/>
-  <joint name="box_2_joint" type="fixed">
+  <xacro:panda_arm arm_id="$(arg arm_id_1)" connected_to="base_link"  xyz="0.0 0.0 0.0" safety_distance="0"/>
+  <joint name="grasp_point_joint" type="fixed">
     <origin rpy="0 0 0" xyz="0.0 0.0 0.0"/>
     <parent link="$(arg arm_id_1)_link8"/>
